File: busdisplay_r2.sch (KiCad schematic (older format))
At the start: 30 parts, among them J1 Hex/Dec, J2 ICSP, J3 Input, J4 Power, Q1 AO3401A, Q2 AO3401A, Q3 AO3401A, U1 PIC16F57-ISO, U2 74HCT245, Y1 8MHz

Commit message: Revision 3 files
Parts:
- removed C4: 15pF, Capacitor_SMD:C_0603_1608Metric, symbol Device:C_Small
- removed JP1: ~PROG~/RUN, Resistor_SMD:R_0603_1608Metric, symbol Device:Jumper_NC_Small
- removed R14: 10k, Resistor_SMD:R_0603_1608Metric, symbol Device:R_Small
- removed U1: PIC16F57-ISO, Package_SO:SOIC-28W_7.5x17.9mm_P1.27mm, symbol busdisplay_r2:PIC16F57-ISO
- removed Y1: 8MHz, Crystal:Crystal_SMD_5032-2Pin_5.0x3.2mm, symbol Device:Crystal_Small
- added U1: PIC16F570-ISO, Package_SO:SOIC-28W_7.5x17.9mm_P1.27mm, symbol busdisplay_r2:PIC16F570-ISO
- C3: value 15pF -> 47uF; footprint Capacitor_SMD:C_0603_1608Metric -> Capacitor_SMD:C_1206_3216Metric
Connections:
- net +5V: now also C3.1, U1.20 (Vdd)
- net A: now also U1.12 (RC1)
- net B: now also U1.14 (RC3)
- net BUF0: now also U1.2 (PA0)
- net BUF1: now also U1.3 (PA1)
- net BUF2: now also U1.4 (PA2)
- net BUF3: now also U1.5 (PA3)
- net BUF4: now also U1.6 (PA4)
- net BUF5: now also U1.7 (PA5)
- net BUF6: now also U1.10 (PA6); no longer J2.5 (Pin_5)
- net BUF7: now also U1.9 (PA7); no longer J2.4 (Pin_4)
- net C: now also U1.17 (RC6)
- net D: now also U1.15 (RC4)
- net DIG1: now also U1.26 (RB5)
- net DIG2: now also U1.25 (RB4)
- net DIG3: now also U1.24 (RB3)
- net DP: now also U1.18 (RC7)
- net E: now also U1.11 (RC0)
- net F: now also U1.13 (RC2)
- net G: now also U1.16 (RC5)
- net GND: now also U2.19 (CE), U1.19 (Vss), U1.8 (Vss)
- net ~MCLR: now also U1.1 (~MCLR~/Vpp)
- net at J1.2 (Pin_2), R2.2: now also U1.21 (RB0)
- new net: J2.4 (Pin_4), U1.28 (RB7/ICSPDAT)
- new net: J2.5 (Pin_5), U1.27 (RB6/ICSPCLK)
- no-connect marks 1 -> 2
Other:
- note removed: "Clear solder bridge to\nenable ICSP"
- moved on the sheet: J1, J2, R2
