File: busdisplay_r2.kicad_pcb (KiCad board)
At the start: 2 copper layers, 35 x 53 mm, 31 parts, among them J1 Hex/Dec, J2 ICSP, J3 Input, J4 Power, Q1 AO3401A, Q2 AO3401A, Q3 AO3401A, U1 PIC16F57-ISO, U2 74HCT245, Y1 8MHz

Commit message: Revision 3 files
Parts:
- removed C4: 15pF, Capacitor_SMD:C_0603_1608Metric
- removed JP1: ~PROG~/RUN, Resistor_SMD:R_0603_1608Metric
- removed R14: 10k, Resistor_SMD:R_0603_1608Metric
- removed Y1: 8MHz, Crystal:Crystal_SMD_5032-2Pin_5.0x3.2mm
- C3: value 15pF -> 47uF; footprint Capacitor_SMD:C_0603_1608Metric -> Capacitor_SMD:C_1206_3216Metric
- U1: value PIC16F57-ISO -> PIC16F570-ISO
- moved C3 35.6 mm to (62.2, 77.8), turned to 0 degrees
- moved J1 29.9 mm to (65.7, 58.5)
- moved J4 29.9 mm to (65.7, 68.6)
- moved Q1 29.1 mm to (37.3, 68.9), turned to 180 degrees
- moved Q3 28.7 mm to (37.3, 76.3), turned to 180 degrees
- moved Q2 28.0 mm to (37.3, 72.6), turned to 180 degrees
- moved J2 27.8 mm to (37.5, 60.5)
- moved G*** 24.2 mm to (62.7, 75.0)
- moved R3 24.0 mm to (40.0, 68.9), turned to 270 degrees
- moved R5 23.5 mm to (40.0, 76.3), turned to 270 degrees
- moved R4 22.6 mm to (40.0, 72.6), turned to 270 degrees
- moved R1 21.9 mm to (40.4, 59.1)
- moved R2 21.2 mm to (61.2, 62.6)
- moved C1 17.2 mm to (52.6, 50.0), turned to 90 degrees
- moved R10 4.06 mm to (61.9, 50.0)
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Connections:
- C3 pad 1: Net-(C3-Pad1) -> +5V
- J2 pad 4: BUF7 -> Net-(J2-Pad4)
- J2 pad 5: BUF6 -> Net-(J2-Pad5)
- U1 pad 1: Net-(U1-Pad1) -> ~MCLR
- U1 pad 10: BUF0 -> BUF6
- U1 pad 11: BUF1 -> E
- U1 pad 12: BUF2 -> A
- U1 pad 13: BUF3 -> F
- U1 pad 14: BUF4 -> B
- U1 pad 15: BUF5 -> D
- U1 pad 16: BUF6 -> G
- U1 pad 17: BUF7 -> C
- U1 pad 18: B -> DP
- U1 pad 19: F -> GND
- U1 pad 2: +5V -> BUF0
- U1 pad 20: A -> +5V
- U1 pad 21: E -> Net-(J1-Pad2)
- U1 pad 22: D -> Net-(U1-Pad22)
- U1 pad 23: G -> Net-(U1-Pad23)
- U1 pad 24: C -> DIG3
- U1 pad 25: DP -> DIG2
- U1 pad 26: Net-(C4-Pad1) -> DIG1
- U1 pad 27: Net-(C3-Pad1) -> Net-(J2-Pad5)
- U1 pad 28: ~MCLR -> Net-(J2-Pad4)
- U1 pad 3: (no net) -> BUF1
- U1 pad 4: GND -> BUF2
- U1 pad 5: (no net) -> BUF3
- U1 pad 6: DIG1 -> BUF4
- U1 pad 7: DIG2 -> BUF5
- U1 pad 8: DIG3 -> GND
- U1 pad 9: Net-(J1-Pad2) -> BUF7
- U2 pad 19: Net-(JP1-Pad1) -> GND
Routing:
- net +5V: track 91.4 -> 118.3 mm, vias 1 -> 0
- net Net-(LED1-Pad12): track 69.0 -> 45.1 mm
- net ~MCLR: track 30.7 -> 7.55 mm
- net Net-(LED1-Pad8): track 48.5 -> 65.6 mm
- net DIG3: track 16.9 -> 28.9 mm
- net BUF0: track 7.97 -> 18.9 mm
- net Net-(JP1-Pad1): track 10.1 -> 0.00 mm
- net BUF1: track 13.4 -> 23.1 mm
- net BUF5: track 19.8 -> 28.9 mm, vias 2 -> 0
- net BUF2: track 15.8 -> 24.6 mm
- net Net-(J2-Pad5): track 0.00 -> 8.46 mm
- net BUF3: track 18.0 -> 26.0 mm
- net D: track 11.1 -> 3.23 mm, vias 2 -> 0
- net G: track 10.9 -> 3.09 mm, vias 2 -> 0
- net DP: track 10.6 -> 2.82 mm, vias 2 -> 0
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Other:
- board text added: "Busdisplay V.3"
- board text added: "LSB"
- board text added: "MSB"
- board text removed: "Busdisplay V.2"
- board text removed: "~PROG~ RUN"

Commit message: Add firmware, gerbers and ibom
Parts:
- removed the G*** at (62.7, 75.0)
- added G***: LOGO, sleepyLogo:sleepylogo_15mm, F.Cu at (50.8, 39.6)
- moved C3 2.99 mm to (60.4, 75.4), turned to 270 degrees
- moved R1 1.63 mm to (40.4, 60.7)
- moved R7 1.40 mm to (65.3, 50.0)
- moved R9 1.40 mm to (58.9, 50.0)
- moved R10 1.40 mm to (60.5, 50.0)
- moved R12 1.40 mm to (57.3, 50.0)
- moved R13 1.40 mm to (54.1, 50.0)
- moved R6 1.40 mm to (62.1, 50.0)
- moved R8 1.40 mm to (55.7, 50.0)
- moved R11 1.40 mm to (63.7, 50.0)
- moved J3 1.14 mm to (42.0, 79.8)
- moved LED1 0.93 mm to (44.5, 46.2)
- moved U2 0.63 mm to (50.9, 72.6)
- moved J1 0.41 mm to (65.3, 58.5)
- moved J4 0.41 mm to (65.3, 68.6)
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Routing:
- net Net-(LED1-Pad8): track 65.6 -> 56.9 mm, vias 0 -> 1
- net Net-(LED1-Pad9): track 57.9 -> 51.8 mm, vias 0 -> 1
- net Net-(LED1-Pad12): track 45.1 -> 40.3 mm, vias 0 -> 1
- net +5V: track 118.3 -> 115.2 mm
- net GND: track 14.5 -> 12.2 mm, vias 6 -> 26
- net BUF7: track 32.1 -> 34.4 mm, vias 2 -> 0
- net Net-(LED1-Pad11): track 27.7 -> 25.8 mm
- net Net-(LED1-Pad10): track 26.5 -> 24.6 mm
- net Net-(LED1-Pad4): track 7.45 -> 5.64 mm
- net Net-(LED1-Pad3): track 8.43 -> 6.63 mm
- net Net-(LED1-Pad1): track 22.5 -> 21.0 mm
- net Net-(LED1-Pad7): track 20.2 -> 18.7 mm
- net Net-(LED1-Pad2): track 17.5 -> 16.2 mm
- net Net-(LED1-Pad5): track 6.07 -> 5.03 mm
- net ~MCLR: track 7.55 -> 6.64 mm
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Other:
- board size 35 x 53 mm -> 33 x 50 mm
- board text added: "Busdisplay Rev.3"
- board text added: "www.sleepyponylabs.com"
- board text removed: "Busdisplay V.3"
- board text removed: "sleepyponylabs.com"
